File: kicad/ahmygroin.kicad_pcb (KiCad board)
At the start: 2 copper layers, 90 x 70 mm, 25 parts, among them J1 BAT, J10 MODE_CON3, J2 BTN, J3 SPK, J4 PROMINI_L, J5 PROMINI_R, J6 SV17F_IO, J7 SV17F_PWR, J8 MODE_CON1, J9 MODE_CON2, Q1 AO3401A, Q3 AO3401A, Q4 MMBT3904

Commit message: v3 PCB re-spin: fix six v2 layout bugs
Build script: kicad/build_v3.py — single-shot transformation from v2
to v3. Idempotent; rolls back via `git reset` to the pre-v3 commit.

Structural fixes (DY-SV17F footprint bug + 5 others, all documented
in PINOUTS.md):

  1-3. DY-SV17F J6/J7 footprints now 1×9 pads each, 2.5 mm metric
       pin pitch (overridden at build time from the stock 2.54 mm
       PinHeader_1x09 footprint), 20.5 mm row pitch. Pin assignments
       per PINOUTS.md (left: SPK+/SPK-/DACL/DACR/V33/V5/CON3-BUSY/
       CON2/CON1; right: TX/RX-trigger/IO2-7/GND).
  4. /CON1, /CON2, /CON3 nets now connect J8/J9/J10 middle pins to
     the J6 footprint in the netlist (v2 had no such connections).
  5. Pro Mini J5 power: /VSYS on pad 1 (RAW), /V33 on pad 4 (VCC).
     Pad 11/12 (D10/D11) un-assigned. v2 had these reversed.
  6. J1 (battery) and J3 (speaker) get '+'/'-' silkscreen markers,
     prepended via sexpdata after pcbnew.SaveBoard (the pcbnew
     PCB_TEXT API produces files that fail to re-load on this
     SWIG build).

Plus: TP1 V33 test point added near C2/C3 cluster; C4 relocated
from (60, 14) to (50, 40) to clear the new DY-SV17F footprint;
C5/C6 moved to (60, 30) and (64, 30); board outline + GND zones
regenerated.

Docs:
- PINOUTS.md: updated U2 form factor (2.5 mm metric pitch, 20.5
  mm row pitch); v3 design-rationale section replaces the v2 errata
  list; added a "v3 routing TBD" note.
- SOLDERING_GUIDE.md: hardware erratum section wrapped in <details>
  collapse with a "v3 status" preface at the top noting the v2 bugs
  are fixed; inline "Errata-revised" callouts in Steps 4/5/7/11.2
  left in place but marked as v2-only context.
- v2/README.md: §3 corrected (DIP-18 / 2.5 mm / 20.5 mm); pin map
  diagram replaced with the 2-column 1×9 layout.

What is NOT done (v3 routing):
- The PCB ships unrouted (76 nets at the ratsnest stage). The v2
  routing in layout_pipeline.py doesn't fit v3 placements; deferred
  to KiCad GUI autorouter or hand-r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
Parts:
- added TP1: V33, TestPoint_THTPad_D1.5mm_Drill0.7mm, F.Cu at (43.0, 40.0)
- J6, J7: footprint PinHeader_1x08_P2.54mm_Vertical -> PinHeader_1x09_P2.54mm_Vertical
- moved C4 27.9 mm to (50.0, 40.0)
- moved C5 27.8 mm to (60.0, 30.0)
- moved C6 22.2 mm to (64.0, 30.0)
- moved J7 2.72 mm to (75.5, 5.00)
Connections:
- J5 pad 1: (no net) -> /VSYS
- J5 pad 11: /V33 -> (no net)
- J5 pad 12: /VSYS -> (no net)
- J5 pad 4: (no net) -> /V33
- J6 pad 1: (no net) -> /SPK_P
- J6 pad 2: /TRIG_OUT -> /SPK_N
- J6 pad 5: (no net) -> /V33
- J6 pad 6: (no net) -> /VDFP
- J6 pad 7: (no net) -> /BUSY_IN
- J6 pad 8: (no net) -> /CON2
- J7 pad 2: /VDFP -> /TRIG_OUT
- J7 pad 3: /GND -> (no net)
- J7 pad 5: /BUSY_IN -> (no net)
- J7 pad 7: /SPK_N -> (no net)
- J7 pad 8: /SPK_P -> (no net)
Routing:
- net /BUSY_IN: track 76.0 -> 0.00 mm
- net /V33: track 74.9 -> 0.00 mm, vias 1 -> 0
- net /VSYS: track 70.0 -> 0.00 mm
- net /BTN_IN: track 63.8 -> 0.00 mm
- net /TRIG_OUT: track 60.8 -> 0.00 mm
- net /SPK_N: track 55.5 -> 0.00 mm
- net /VDFP: track 54.0 -> 0.00 mm
- net /SPK_P: track 41.4 -> 0.00 mm
- net /Q4_BASE: track 15.6 -> 0.00 mm
- net /Q1_GATE: track 14.1 -> 0.00 mm
- net /GATE_CTRL: track 12.8 -> 0.00 mm
- net /VBATT: track 7.11 -> 0.00 mm
Other:
- board text added: "+"
- board text added: "-"
- board text added: "V33"

Commit message: v3.1 PCB: fix mode-select, IO0 trigger, CON3 pull-down
Three bugs uncovered during v2 board bring-up (audio was silent):

1. CON1/CON2/CON3 mode table was wrong. The docs called for
   CON1=GND, CON2=V33, CON3=floating, which is not a valid mode
   per the DY-SV17F datasheet. Correct mode for "ground IO0 plays
   00001.mp3" is I/O Independent Mode 0: CON1=GND, CON2=V33,
   CON3=GND.

2. /TRIG_OUT was routed to J7 pad 2 (= module RX/IO1). In
   Independent Mode 0, IO1 plays 00002.mp3, not 00001.mp3. The
   correct pin for track 1 is IO0 (right pin 1).

3. Firmware D7 INPUT_PULLUP pulled CON3 HIGH during the chip's
   first-30ms mode-sample, silently switching modes. Firmware
   now uses D7 INPUT (no pullup) and a fixed playback delay
   instead of BUSY polling.

v3 PCB changes (build_v3.py + ahmygroin.kicad_pcb + .net):
  - /TRIG_OUT moved from J7 pad 2 to J7 pad 1 (IO0)
  - /CON3 net folded into /BUSY_IN; J10 pad 2 now reaches the
    module CON3/BUSY pin via the BUSY_IN wiring
  - R3 (10 kOhm 0805) added as CON3 pull-down to GND, so the
    chip samples CON3=LOW at boot while the push-pull BUSY
    output can still drive the line HIGH afterwards
  - J1 / J3 polarity silkscreen moved to -5 mm offset to clear
    the connector body silk outlines

Verification (KiCad MCP + kicad-cli):
  27 footprints, 101 tracks, 2 vias, GND zones filled on both
  copper layers. Freerouting v2.0.1 (Java 21) autoroute. DRC:
  0 violations, 0 unconnected items.

Docs synced: PINOUTS.md (real CON1/2/3 truth table + Mode 0
setup), SOLDERING_GUIDE.md (mode-select rewrite, wire #1 to
IO0, D7-no-pullup gotcha, 5-digit 00001.mp3 filename),
v2/README.md, v2/bom.md, PLANS.md.

Firmware: v2/firmware/main.cpp updated for IO0 + fixed-delay
playback. v2/firmware/main.cpp.bak removed (obsolete).

Schematic redo (kicad/ahmygroin.kicad_sch) deferred. The
schematic uses 8-pin Conn_01x08 symbols and pre-v3.1 labels;
build_v3.py mutates the netlist directly, so PCB+netlist are
the source of truth for fab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
Parts:
- added R3: 10k, R_0805_2012Metric, F.Cu at (62.0, 46.0)
Connections:
- J10 pad 2: /CON3 -> /BUSY_IN
- J7 pad 1: (no net) -> /TRIG_OUT
- J7 pad 2: /TRIG_OUT -> (no net)
Routing:
- net /V33: track 0.00 -> 93.6 mm
- net /VSYS: track 0.00 -> 89.2 mm
- net /BUSY_IN: track 0.00 -> 88.5 mm
- net /TRIG_OUT: track 0.00 -> 83.5 mm, vias 0 -> 1
- net /SPK_N: track 0.00 -> 66.3 mm
- net /SPK_P: track 0.00 -> 66.0 mm
- net /BTN_IN: track 0.00 -> 50.2 mm
- net /VDFP: track 0.00 -> 38.7 mm, vias 0 -> 1
- net /CON1: track 0.00 -> 31.4 mm
- net /CON2: track 0.00 -> 28.6 mm
- net /Q4_BASE: track 0.00 -> 15.3 mm
- net /Q1_GATE: track 0.00 -> 13.9 mm
- net /GATE_CTRL: track 0.00 -> 10.6 mm
- net /VBATT: track 0.00 -> 7.08 mm

Commit message: v3.2 PCB: solder-and-go board, no flying wires
The v2 board needed twelve hand-soldered wires and still idled at 14 mA.
This respin makes the next board work from the bag of parts alone.

Electrical fixes (kicad/build_v3.py):

* Split /V33. The Pro Mini's always-on VCC (J5.4) no longer touches the
  mode-select jumper rail; the rail is fed only by the DY-SV17F's own
  gated V33 output. This is the CON2 phantom-power path -- 8.7 mA of
  permanent idle draw, closed in copper.
* Re-orient Q3. Drain now faces the battery and source the load. It was
  backwards, meaning v2 and v3.1 had a reverse-polarity FET fitted and no
  reverse-polarity protection.
* Bond the Pro Mini's second ground (J5.2).

Placement: nothing sits under either module body any more. R1, C2, C3 and
TP1 were evicted. KiCad DRC cannot catch this class of bug -- pin-header
courtyards cover the header strip, not the module that overhangs it -- so
it is now asserted geometrically instead.

Silkscreen: chamfered body outlines for both modules, all 42 module pin
names, jumper settings printed next to each jumper, connector names and
polarity, and a board title carrying the idle-current figure.

Routing: fully autorouted headless. 148 tracks/vias, 2 filled zones,
0 unconnected, 0 DRC violations.

New tooling:

* kicad/verify_v3.py -- the pre-fab gate. Checks module-body keep-outs,
  the electrical assertions above, silk-over-pad, and routing
  completeness. Exit 0 only on PASS. Run it before ordering.
* kicad/route_v3.py -- DSN -> Freerouting -> SES -> fill. Exports a
  zone-free copy so Freerouting routes GND as real copper rather than
  assuming a poured plane and skipping it; runs each pcbnew step in its
  own process because chaining them degrades the SWIG board handle.

Docs: SOLDERING_GUIDE.md rewritten for v3.2 -- headers belong to the
modules, Step 7 is "plug both in", the 1:1 paper fit check is now a
mandatory gate, and the continuity checks are grouped and re-derived
against module pins. PINOUTS.md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
Parts:
- moved C2 15.3 mm to (20.0, 43.0)
- moved C3 15.3 mm to (24.0, 43.0)
- moved R1 13.7 mm to (38.0, 34.0)
- moved R3 5.00 mm to (62.0, 41.0)
- moved C5 4.24 mm to (57.0, 33.0)
- moved TP1 4.12 mm to (44.0, 44.0)
- moved C6 3.61 mm to (62.0, 33.0)
- moved R2 1.00 mm to (45.0, 34.0)
Connections:
- J5 pad 2: (no net) -> /GND
- J5 pad 4: /V33 -> (no net)
- Q3 pad 2: /VBATT -> /VSYS
- Q3 pad 3: /VSYS -> /VBATT
Routing:
- net /GND: track 0.00 -> 302.7 mm, vias 0 -> 1
- net /V33: track 93.6 -> 64.0 mm
- net /VSYS: track 89.2 -> 110.0 mm
- net /GATE_CTRL: track 10.6 -> 30.3 mm
- net /TRIG_OUT: track 83.5 -> 70.2 mm, vias 1 -> 0
- net /Q4_BASE: track 15.3 -> 5.80 mm
- net /VDFP: track 38.7 -> 46.3 mm, vias 1 -> 0
- net /BUSY_IN: track 88.5 -> 91.4 mm
- net /VBATT: track 7.08 -> 8.80 mm
Other:
- board text added: "A0"
- board text added: "A1"
- board text added: "A2"
- board text added: "A3"
- board text added: "AH! MY GROIN! v3.2"
- board text added: "BATTERY"
- board text added: "BUSY"
- board text added: "BUTTON"
- board text added: "CON1"
- board text added: "CON2"
- board text added: "CON3"
- board text added: "D10"
- board text added: "D11"
- board text added: "D12"
- board text added: "D13"
- board text added: "D2"
- board text added: "D3"
- board text added: "D4"
- board text added: "D5"
- board text added: "D6"
- board text added: "D7"
- board text added: "D8"
- board text added: "D9"
- board text added: "DACL"
- board text added: "DACR"
- board text added: "DY-SV17F"
- board text added: "GND"
- board text added: "IDLE 0.15mA - NO WIRE LINKS"
- board text added: "IO0"
- board text added: "IO1"
- board text added: "IO2"
- board text added: "IO3"
- board text added: "IO4"
- board text added: "IO5"
- board text added: "IO6"
- board text added: "IO7"
- board text added: "NO SHUNT"
- board text added: "PRO MINI"
- board text added: "RAW"
- board text added: "RST"
- board text added: "RXI"
- board text added: "SHUNT 1-2"
- board text added: "SHUNT 2-3"
- board text added: "SPEAKER"
- board text added: "SPK+"
- board text added: "SPK-"
- board text added: "TXO"
- board text added: "V5"
- board text added: "VCC"
